File: ID.kicad_sch (KiCad schematic)
At the start: 25 parts

Commit message: assembly
Parts:
- R?: fit_field (none) -> DNP
Changed lines of the file:
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@@
-(kicad_sch (version 20230121) (generator eeschema)
+(kicad_sch (version 20230409) (generator eeschema)
   (paper "A3")
   (title_block

Commit message: - zero origin on so - silk - sch trig and rtsi lines need 510 resistor - assembly updated - sch and pcb project name and rev - no changes to gerber, old one can be used
Other:
- title: EOL ECU POWER CARD -> EOL ECU MIX CARD
Changed lines of the file:
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@@
   (paper "A3")
   (title_block
-    (title "EOL ECU POWER CARD")
-    (date "2023-04-03")
-    (rev "0B")
+    (title "EOL ECU MIX CARD")
+    (date "2023-09-26")
+    (rev "0C")
     (company "ARXTRON TECHNOLOGIES")
     (comment 1 "A0180-V0")

Commit message: pnp added
Parts:
- R?: now left out of the parts list
Changed lines of the file:
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@@
-(kicad_sch (version 20230620) (generator eeschema)
+(kicad_sch (version 20230819) (generator eeschema)
   (paper "A3")
   (title_block
