File: load.kicad_sch (KiCad schematic)
At the start: 49 parts, among them K1 G6K-2G-Y-TR_DC24_DPDT, K10 G6K-2G-Y-TR_DC24_DPDT, K11 G6K-2G-Y-TR_DC24_DPDT, K12 G6K-2G-Y-TR_DC24_DPDT, K13 G6K-2G-Y-TR_DC24_DPDT, K14 G6K-2G-Y-TR_DC24_DPDT, K15 G6K-2G-Y-TR_DC24_DPDT, K16 G6K-2G-Y-TR_DC24_DPDT, K2 G6K-2G-Y-TR_DC24_DPDT, K3 G6K-2G-Y-TR_DC24_DPDT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

Commit message: - zero origin on so - silk - sch trig and rtsi lines need 510 resistor - assembly updated - sch and pcb project name and rev - no changes to gerber, old one can be used
Other:
- title: EOL ECU POWER CARD -> EOL ECU MIX CARD
Changed lines of the file:
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@@
   (paper "A3")
   (title_block
-    (title "EOL ECU POWER CARD")
-    (date "2023-04-03")
-    (rev "0B")
+    (title "EOL ECU MIX CARD")
+    (date "2023-09-26")
+    (rev "0C")
     (company "ARXTRON TECHNOLOGIES")
     (comment 1 "A0180-V0")
