File: load.kicad_sch (KiCad schematic)
At the start: 49 parts, among them K1 G6K-2G-Y-TR_DC24_DPDT, K10 G6K-2G-Y-TR_DC24_DPDT, K11 G6K-2G-Y-TR_DC24_DPDT, K12 G6K-2G-Y-TR_DC24_DPDT, K13 G6K-2G-Y-TR_DC24_DPDT, K14 G6K-2G-Y-TR_DC24_DPDT, K15 G6K-2G-Y-TR_DC24_DPDT, K16 G6K-2G-Y-TR_DC24_DPDT, K2 G6K-2G-Y-TR_DC24_DPDT, K3 G6K-2G-Y-TR_DC24_DPDT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

Commit message: kicad 9 - r11-check gerber before sending to manufacturing
Parts:
- gave numbers to parts that had none: 32

Commit message: r11a - clean up mostly with reports naming, values, footprints and parts
Other:
- company: ARXTRON TECHNOLOGIES -> ${COMPANY}
- title: EOL ECU MIX CARD -> ${PART_NUM} ${PCB_NAME} ${ASSY_VARIANT} ${ASSY_NAME}
Changed lines of the file:
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@@
 	(paper "A3")
 	(title_block
-		(title "EOL ECU MIX CARD")
-		(date "2023-09-26")
-		(rev "0C")
-		(company "ARXTRON TECHNOLOGIES")
-		(comment 1 "A0180-V0")
-		(comment 2 "PRJ22180")
-		(comment 3 "EOL ECU RCM8 RCM9")
-		(comment 4 "ANTON TOKARSKYI")
+		(title "${PART_NUM} ${PCB_NAME} ${ASSY_VARIANT} ${ASSY_NAME}")
+		(date "2025-03-12")
+		(rev "${REVISION}${REVISION_SCH}")
+		(company "${COMPANY}")
+		(comment 1 "${PART_NUM}")
+		(comment 2 "${PRJ_NUM}")
+		(comment 3 "${PRJ_NAME}")
+		(comment 4 "${DESIGNED}")
+		(comment 5 "${PART_NUM_ICT}")
 	)
 	(junction
