File: output_n.kicad_sch (KiCad schematic)
At the start: 23 parts

Commit message: kicad 9 - r11-check gerber before sending to manufacturing
Parts:
- C37: renamed from C?; Nominal 0.1µF -> 0.1uF; SupllierPartNumber 478-3352-1-ND -> (none)
- IC4: renamed from IC?; SupllierPartNumber MCP23S17-E/SO-ND -> (none)
- MH5: renamed from MH3; now left out of the parts list
- MH6: renamed from MH4; now left out of the parts list
- R117, R118, R119, R120, R122, R125, R126, R127, R128, R129, R130, R131, R133, R134, R135, R136, R137, R138: renamed from R?; SupllierPartNumber 311-4.7KARCT-ND -> (none); Tolerance 5% -> (none)
- R124: renamed from R?; SupllierPartNumber 311-1.00KCRCT-ND -> (none); Tolerance 1% -> (none)
Connections:
- net GNDD renamed GND_3V3

Commit message: r11a - clean up mostly with reports naming, values, footprints and parts
Other:
- company: ARXTRON TECHNOLOGIES -> ${COMPANY}
- title: EOL ECU MIX CARD -> ${PART_NUM} ${PCB_NAME} ${ASSY_VARIANT} ${ASSY_NAME}
Changed lines of the file:
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@@
 	(paper "A3")
 	(title_block
-		(title "EOL ECU MIX CARD")
-		(date "2023-09-26")
-		(rev "0C")
-		(company "ARXTRON TECHNOLOGIES")
-		(comment 1 "A0180-V0")
-		(comment 2 "PRJ22180")
-		(comment 3 "EOL ECU RCM8 RCM9")
-		(comment 4 "ANTON TOKARSKYI")
+		(title "${PART_NUM} ${PCB_NAME} ${ASSY_VARIANT} ${ASSY_NAME}")
+		(date "2025-03-12")
+		(rev "${REVISION}${REVISION_SCH}")
+		(company "${COMPANY}")
+		(comment 1 "${PART_NUM}")
+		(comment 2 "${PRJ_NUM}")
+		(comment 3 "${PRJ_NAME}")
+		(comment 4 "${DESIGNED}")
+		(comment 5 "${PART_NUM_ICT}")
 	)
 	(text "TODO:\n\n- INTERRUPT OUTPUT CAN BE CONFIGURED AS ACTIVE-HIGH, ACTIVE-LOW OR OPEN-DRAIN\n - VSUP (FOR RELAY'S COIL ...) AND 3V3 (MICROCONTROLLER, MCP ...)\n\n\n\n"
