File: input.kicad_sch (KiCad schematic)
At the start: 89 parts, among them U18 TLP290-4(TPE, U19 TLP290-4(TPE, U20 TLP290-4(TPE, U21 TLP290-4(TPE

Commit message: assy
Parts:
- R? (x2): value RC0603JR-072K2L -> RC0603FR-07510RL; symbol Resistor_Yageo:RC0603JR-072K2L -> Resistor_Yageo:RC0603FR-07510RL; ManufacturerPartNumber RC0603JR-072K2L -> RC0603FR-07510RL; Nominal 2.2k -> 510; SupplierPartNumber 311-2.2KGRCT-ND -> 311-510HRCT-ND

Commit message: - zero origin on so - silk - sch trig and rtsi lines need 510 resistor - assembly updated - sch and pcb project name and rev - no changes to gerber, old one can be used
Other:
- title: EOL ECU POWER CARD -> EOL ECU MIX CARD
Changed lines of the file:
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@@
   (paper "A3")
   (title_block
-    (title "EOL ECU POWER CARD")
-    (date "2023-04-03")
-    (rev "0B")
+    (title "EOL ECU MIX CARD")
+    (date "2023-09-26")
+    (rev "0C")
     (company "ARXTRON TECHNOLOGIES")
     (comment 1 "A0180-V0")

Commit message: wip res
Parts:
- R? (x2): now not fitted; now left out of the parts list
