File: input.kicad_sch (KiCad schematic)
At the start: 89 parts, among them U18 TLP290-4(TPE, U19 TLP290-4(TPE, U20 TLP290-4(TPE, U21 TLP290-4(TPE

Commit message: kicad 9 - r11-check gerber before sending to manufacturing
Parts:
- C38, C39, C40, C41, C42, C43, C45, C47, C48, C53, C55, C57, C61, C63, C66, C68: Nominal 0.1µF -> 0.1uF; SupllierPartNumber 478-3352-1-ND -> (none)
- C69: renamed from C?; Nominal 0.1µF -> 0.1uF; SupllierPartNumber 478-3352-1-ND -> (none)
- IC2: renamed from IC?; SupllierPartNumber MCP23S17-E/SO-ND -> (none)
- R132, R187, R189, R190, R191, R192, R193, R194, R219, R220, R223, R224, R225, R226, R227, R228: SupllierPartNumber 311-2.2KERCT-ND -> (none)
- R188: SupllierPartNumber 311-1.00KCRCT-ND -> (none); Tolerance 1% -> (none)
- R195, R196, R197, R198, R199, R200, R201, R202, R221, R222, R229, R230, R231, R232, R233, R234, R235, R236: SupllierPartNumber 311-4.7KARCT-ND -> (none); Tolerance 5% -> (none)
- R211, R212: renamed from R?; Tolerance 5% -> (none)
- U18, U19, U20, U21: footprint _SOIC_SOP:SOIC127P600X126-16 -> _SOIC_SOP:SOIC127P700X220-16
- gave numbers to parts that had none: 22
Connections:
- net GNDD renamed GND_3V3
Changed lines of the file:
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@@
-(kicad_sch (version 20230819) (generator eeschema)
-  (paper "A3")
-  (title_block
-    (title "EOL ECU MIX CARD")
-    (date "2023-09-26")
-    (rev "0C")
-    (company "ARXTRON TECHNOLOGIES")
-    (comment 1 "A0180-V0")
-    (comment 2 "PRJ22180")
-    (comment 3 "EOL ECU RCM8 RCM9")
-    (comment 4 "ANTON TOKARSKYI")
-  )
+(kicad_sch
+	(version 20250114)
+	(generator "eeschema")
+	(generator_version "9.0")
+	(paper "A3")
+	(title_block
+		(title "EOL ECU MIX CARD")
+		(date "2023-09-26")
+		(rev "0C")
+		(company "ARXTRON TECHNOLOGIES")
+		(comment 1 "A0180-V0")
+		(comment 2 "PRJ22180")
+		(comment 3 "EOL ECU RCM8 RCM9")
+		(comment 4 "ANTON TOKARSKYI")
+	)

Commit message: r11a - clean up mostly with reports naming, values, footprints and parts
Other:
- company: ARXTRON TECHNOLOGIES -> ${COMPANY}
- title: EOL ECU MIX CARD -> ${PART_NUM} ${PCB_NAME} ${ASSY_VARIANT} ${ASSY_NAME}
Changed lines of the file:
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@@
 	(paper "A3")
 	(title_block
-		(title "EOL ECU MIX CARD")
-		(date "2023-09-26")
-		(rev "0C")
-		(company "ARXTRON TECHNOLOGIES")
-		(comment 1 "A0180-V0")
-		(comment 2 "PRJ22180")
-		(comment 3 "EOL ECU RCM8 RCM9")
-		(comment 4 "ANTON TOKARSKYI")
+		(title "${PART_NUM} ${PCB_NAME} ${ASSY_VARIANT} ${ASSY_NAME}")
+		(date "2025-03-12")
+		(rev "${REVISION}${REVISION_SCH}")
+		(company "${COMPANY}")
+		(comment 1 "${PART_NUM}")
+		(comment 2 "${PRJ_NUM}")
+		(comment 3 "${PRJ_NAME}")
+		(comment 4 "${DESIGNED}")
+		(comment 5 "${PART_NUM_ICT}")
 	)
