File: power.kicad_sch (KiCad schematic)
At the start: 55 parts, among them U2 TLP290-4(TPE, U23 LT3060ETS8-5#TRMPBF, U28 ACSL-6210-00RE, U30 NLVVHC1G126DFT1G

Commit message: kicad 9 - r11-check gerber before sending to manufacturing
Parts:
- C2, C81, C90: renamed from C31; Nominal 0.1µF -> 0.1uF
- C26, C27, C29: SupllierPartNumber 1276-3387-1-ND -> (none)
- C28: SupllierPartNumber 478-7476-1-ND -> (none)
- C3, C7: Nominal 0.1µF -> 0.1uF; SupllierPartNumber 478-3352-1-ND -> (none)
- C4, C5, C6: renamed from C32; Nominal 0.1µF -> 0.1uF; SupllierPartNumber 478-3352-1-ND -> (none)
- C83: renamed from C75; Nominal 0.1µF -> 0.1uF
- C87: renamed from C77; Nominal 0.1µF -> 0.1uF
- L2: SupllierPartNumber 1951-1047-ND -> (none)
- PWR1: SupllierPartNumber TDN3-2410WISM-ND -> (none); SupplierDevicePackage 7-SMD Module 6 Leads -> (none)
- R142, R143, R153, R154: renamed from R?; Tolerance 5% -> (none)
- R144, R145, R155: renamed from R219; SupllierPartNumber 311-2.2KERCT-ND -> (none)
- R149, R151: renamed from R191; SupllierPartNumber 311-2.2KERCT-ND -> (none)
- U26: renamed from U2; footprint _SOIC_SOP:SOIC127P600X126-16 -> _SOIC_SOP:SOIC127P700X220-16
- VR1: SupllierPartNumber 495-7459-1-ND -> (none)
- gave numbers to parts that had none: 5
- renumbered C1 to C59, C44 to C82, C50 to C84, C51 to C85, C52 to C86, C80 to C88, C1 to C89, DS37 to DS38, R151 to R148, R151 to R150, R14 to R152, R18 to R282, R113 to R283, R151 to R284, R18 to R308, U23 to U29
Connections:
- net GNDD renamed GND_3V3
- net GND_SIGNAL renamed GND_SIM
Changed lines of the file:
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@@
-(kicad_sch (version 20230819) (generator eeschema)
-  (paper "A3")
-  (title_block
-    (title "EOL ECU MIX CARD")
-    (date "2023-09-26")
-    (rev "0C")
-    (company "ARXTRON TECHNOLOGIES")
-    (comment 1 "A0180-V0")
-    (comment 2 "PRJ22180")
-    (comment 3 "EOL ECU RCM8 RCM9")
-    (comment 4 "ANTON TOKARSKYI")
-  )
+(kicad_sch
+	(version 20250114)
+	(generator "eeschema")
+	(generator_version "9.0")
+	(paper "A3")
+	(title_block
+		(title "EOL ECU MIX CARD")
+		(date "2023-09-26")
+		(rev "0C")
+		(company "ARXTRON TECHNOLOGIES")
+		(comment 1 "A0180-V0")
+		(comment 2 "PRJ22180")
+		(comment 3 "EOL ECU RCM8 RCM9")
+		(comment 4 "ANTON TOKARSKYI")
+	)

Commit message: r11a - clean up mostly with reports naming, values, footprints and parts
Parts:
- added unit 1 of D1
Connections:
- no-connect marks 6 -> 8
Other:
- company: ARXTRON TECHNOLOGIES -> ${COMPANY}
- title: EOL ECU MIX CARD -> ${PART_NUM} ${PCB_NAME} ${ASSY_VARIANT} ${ASSY_NAME}
- moved on the sheet: C82, C83, C84, C85, C86, C87, C88, DS38, R282, R283
Changed lines of the file:
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@@
 	(paper "A3")
 	(title_block
-		(title "EOL ECU MIX CARD")
-		(date "2023-09-26")
-		(rev "0C")
-		(company "ARXTRON TECHNOLOGIES")
-		(comment 1 "A0180-V0")
-		(comment 2 "PRJ22180")
-		(comment 3 "EOL ECU RCM8 RCM9")
-		(comment 4 "ANTON TOKARSKYI")
+		(title "${PART_NUM} ${PCB_NAME} ${ASSY_VARIANT} ${ASSY_NAME}")
+		(date "2025-03-12")
+		(rev "${REVISION}${REVISION_SCH}")
+		(company "${COMPANY}")
+		(comment 1 "${PART_NUM}")
+		(comment 2 "${PRJ_NUM}")
+		(comment 3 "${PRJ_NAME}")
+		(comment 4 "${DESIGNED}")
+		(comment 5 "${PART_NUM_ICT}")
 	)
